File: kratos_week2/week2_q3/week2_q3.kicad_pcb (KiCad board)
At the start: 2 copper layers, 240 x 145.5 mm, 17 parts, among them J1 XT60-M, J10 XT60-M, J11 XT60-M, J2 XT60-M, J3 XT60-M, J4 XT60-M, J5 XT60-M, J6 XT60-M, J7 Conn_01x02_Pin, J8 Conn_01x02_Pin, J9 Conn_01x02_Pin

Commit message: Week2_update
Parts:
- J1, J2, J3, J4, J5, J6: value XT60-M -> XT60PW-F; footprint Connector_AMASS:AMASS_XT60-M_1x02_P7.20mm_Vertical -> Xt60:CONN_XT60PW-F_AMA
- moved J6 8.60 mm to (108.5, 141.6)
- moved J5 8.17 mm to (137.7, 141.6)
- moved J4 7.79 mm to (166.9, 141.4)
- moved J3 7.36 mm to (196.1, 141.4)
- moved J2 6.94 mm to (225.3, 141.4)
- moved J1 6.46 mm to (254.5, 141.6)
Routing:
- net /Vo_11.1V: track 160.3 -> 148.2 mm
- net GND: track 553.8 -> 562.4 mm
- net /Vo_20V: track 237.2 -> 229.2 mm
